File: hardware/SGTL5000.sch (KiCad schematic (older format))
At the start: 24 parts, among them J2 AudioJack3_Ground, J3 AudioJack3_Ground, U2 MCP1811A, U7 SGTL5000

Commit message: fix wiring & routing for lrclk and bclk, and removed lp filter behind pot mux
Other:
- note removed: "these were mislabelled in the symbol\n"
Changed lines of the file:
@@
 encoding utf-8
 Sheet 2 3
-Title ""
-Date ""
-Rev ""
-Comp ""
+Title "teensy-fx"
+Date "2020-02-10"
+Rev "v2"
+Comp "mattvenn"
 Comment1 ""
 Comment2 ""
@@
 Text Notes 4700 1350 0    118  Italic 24
 SGTL5000 audio driver
-Text Notes 2500 3800 0    50   ~ 0
-these were mislabelled in the symbol\n
-$Comp
-L Device:C_Small C?
+$Comp
+L Device:C_Small C?
