File: hardware/pots.sch (KiCad schematic (older format))
At the start: 46 parts, among them SW1 Switch_SW_Push, SW2 Switch_SW_Push, SW3 Switch_SW_Push, SW4 Switch_SW_Push, U4 4067, U5 TLC5947DAP

Commit message: add model number
Other:
- note added: "all pots 10k, taper 1b (linear)\nRK09K1130AP5"
- note removed: "all pots 10k, taper 1b (linear)"
Changed lines of the file:
@@
 RC filter\n200R & 2.2u = 360Hz cutoff
 Text Notes 2200 7300 0    50   ~ 0
-all pots 10k, taper 1b (linear)
+all pots 10k, taper 1b (linear)\nRK09K1130AP5
 Text Notes 2300 7450 0    50   ~ 0
 all pots together = 4mA

Commit message: changed to LDO that I can source from farnell
Parts:
- D1, D10, D11, D12, D13, D14, D15, D16, D17, D18, D19, D2, D20, D3, D4, D5, D6, D7, D8, D9: farnell (none) -> 2099236
Changed lines of the file:
@@
 F 2 "LED_SMD:LED_0805_2012Metric" H 9400 3000 50  0001 C CNN
 F 3 "~" H 9400 3000 50  0001 C CNN
+F 4 "2099236" H 9400 3000 50  0001 C CNN "farnell"
 	1    9400 3000
 	1    0    0    -1
@@
 F 2 "LED_SMD:LED_0805_2012Metric" H 8800 2900 50  0001 C CNN
 F 3 "~" H 8800 2900 50  0001 C CNN
+F 4 "2099236" H 8800 2900 50  0001 C CNN "farnell"
 	1    8800 2900
 	1    0    0    -1
@@
 F 2 "LED_SMD:LED_0805_2012Metric" H 8250 2800 50  0001 C CNN
 F 3 "~" H 8250 2800 50  0001 C CNN
+F 4 "2099236" H 8250 2800 50  0001 C CNN "farnell"
 	1    8250 2800
 	1    0    0    -1
@@
 F 2 "LED_SMD:LED_0805_2012Metric" H 10000 2700 50  0001 C CNN
 F 3 "~" H 10000 2700 50  0001 C CNN
+F 4 "2099236" H 10000 2700 50  0001 C CNN "farnell"
 	1    10000 2700
 	1    0    0    -1
@@
 F 2 "LED_SMD:LED_0805_2012Metric" H 9400 2600 50  0001 C CNN
 F 3 "~" H 9400 2600 50  0001 C CNN
+F 4 "2099236" H 9400 2600 50  0001 C CNN "farnell"
 	1    9400 2600
 	1    0    0    -1
@@
 F 2 "LED_SMD:LED_0805_2012Metric" H 8800 2500 50  0001 C CNN
 F 3 "~" H 8800 2500 50  0001 C CNN
+F 4 "2099236" H 8800 2500 50  0001 C CNN "farnell"
 	1    8800 2500
 	1    0    0    -1
@@
 F 2 "LED_SMD:LED_0805_2012Metric" H 8250 2400 50  0001 C CNN
 F 3 "~" H 8250 2400 50  0001 C CNN
+F 4 "2099236" H 8250 2400 50  0001 C CNN "farnell"
 	1    8250 2400
 	1    0    0    -1
@@
 F 2 "LED_SMD:LED_0805_2012Metric" H 10000 3100 50  0001 C CNN
 F 3 "~" H 10000 3100 50  0001 C CNN
+F 4 "2099236" H 10000 3100 50  0001 C CNN "farnell"
 	1    10000 3100
 	1    0    0    -1
@@
 F 2 "LED_SMD:LED_0805_2012Metric" H 9400 3800 50  0001 C CNN
 F 3 "~" H 9400 3800 50  0001 C CNN
+F 4 "2099236" H 9400 3800 50  0001 C CNN "farnell"
 	1    9400 3800
 	1    0    0    -1
@@
 F 2 "LED_SMD:LED_0805_2012Metric" H 8800 3700 50  0001 C CNN
 F 3 "~" H 8800 3700 50  0001 C CNN
+F 4 "2099236" H 8800 3700 50  0001 C CNN "farnell"
 	1    8800 3700
 	1    0    0    -1
@@
 F 2 "LED_SMD:LED_0805_2012Metric" H 8250 3600 50  0001 C CNN
 F 3 "~" H 8250 3600 50  0001 C CNN
+F 4 "2099236" H 8250 3600 50  0001 C CNN "farnell"
 	1    8250 3600
 	1    0    0    -1
@@
 F 2 "LED_SMD:LED_0805_2012Metric" H 10000 3500 50  0001 C CNN
 F 3 "~" H 10000 3500 50  0001 C CNN
+F 4 "2099236" H 10000 3500 50  0001 C CNN "farnell"
 	1    10000 3500
 	1    0    0    -1
@@
 F 2 "LED_SMD:LED_0805_2012Metric" H 9400 3400 50  0001 C CNN
 F 3 "~" H 9400 3400 50  0001 C CNN
+F 4 "2099236" H 9400 3400 50  0001 C CNN "farnell"
 	1    9400 3400
 	1    0    0    -1
@@
 F 2 "LED_SMD:LED_0805_2012Metric" H 8800 3300 50  0001 C CNN
 F 3 "~" H 8800 3300 50  0001 C CNN
+F 4 "2099236" H 8800 3300 50  0001 C CNN "farnell"
 	1    8800 3300
 	1    0    0    -1
@@
 F 2 "LED_SMD:LED_0805_2012Metric" H 8250 3200 50  0001 C CNN
 F 3 "~" H 8250 3200 50  0001 C CNN
+F 4 "2099236" H 8250 3200 50  0001 C CNN "farnell"
 	1    8250 3200
 	1    0    0    -1
@@
 F 2 "LED_SMD:LED_0805_2012Metric" H 10000 3900 50  0001 C CNN
 F 3 "~" H 10000 3900 50  0001 C CNN
+F 4 "2099236" H 10000 3900 50  0001 C CNN "farnell"
 	1    10000 3900
 	1    0    0    -1
@@
 F 2 "LED_SMD:LED_0805_2012Metric" H 9400 4200 50  0001 C CNN
 F 3 "~" H 9400 4200 50  0001 C CNN
+F 4 "2099236" H 9400 4200 50  0001 C CNN "farnell"
 	1    9400 4200
 	1    0    0    -1
@@
 F 2 "LED_SMD:LED_0805_2012Metric" H 8800 4100 50  0001 C CNN
 F 3 "~" H 8800 4100 50  0001 C CNN
+F 4 "2099236" H 8800 4100 50  0001 C CNN "farnell"
 	1    8800 4100
 	1    0    0    -1
@@
 F 2 "LED_SMD:LED_0805_2012Metric" H 8250 4000 50  0001 C CNN
 F 3 "~" H 8250 4000 50  0001 C CNN
+F 4 "2099236" H 8250 4000 50  0001 C CNN "farnell"
 	1    8250 4000
 	1    0    0    -1
@@
 F 2 "LED_SMD:LED_0805_2012Metric" H 10000 4300 50  0001 C CNN
 F 3 "~" H 10000 4300 50  0001 C CNN
+F 4 "2099236" H 10000 4300 50  0001 C CNN "farnell"
 	1    10000 4300
 	1    0    0    -1

Commit message: farnell numbers
Parts:
- C10, C11, C12, C16: farnell (none) -> 2773238
- L2: farnell (none) -> 2215655
- R10: value 200r -> 100R; farnell (none) -> 1469862
- R4: farnell (none) -> 2906645
- R5: value 5k -> 4.7k; farnell (none) -> 1469923
- RV10, RV11, RV12, RV2, RV3, RV4, RV5, RV6, RV7, RV8, RV9: rs (none) -> 729-3600
- SW1, SW2, SW3, SW4: farnell (none) -> dnp
Other:
- note added: "RC filter\n200R & 2.2u = 700Hz cutoff"
- note removed: "RC filter\n200R & 2.2u = 360Hz cutoff"
Changed lines of the file:
@@
 F 2 "Resistor_SMD:R_0805_2012Metric" V 3380 2300 50  0001 C CNN
 F 3 "~" H 3450 2300 50  0001 C CNN
+F 4 "2906645" H 3450 2300 50  0001 C CNN "farnell"
 	1    3450 2300
 	0    1    1    0
@@
 F 2 "audio-fx:Potentiometer_Alps_RK09L_Single_Vertical" H 2400 4900 50  0001 C CNN
 F 3 "~" H 2400 4900 50  0001 C CNN
+F 4 "729-3600" H 2400 4900 50  0001 C CNN "rs"
 	1    2400 4900
 	1    0    0    -1
@@
 F 2 "audio-fx:Potentiometer_Alps_RK09L_Single_Vertical" H 3150 4900 50  0001 C CNN
 F 3 "~" H 3150 4900 50  0001 C CNN
+F 4 "729-3600" H 3150 4900 50  0001 C CNN "rs"
 	1    3150 4900
 	1    0    0    -1
@@
 F 2 "audio-fx:Potentiometer_Alps_RK09L_Single_Vertical" H 3900 4900 50  0001 C CNN
 F 3 "~" H 3900 4900 50  0001 C CNN
+F 4 "729-3600" H 3900 4900 50  0001 C CNN "rs"
 	1    3900 4900
 	1    0    0    -1
@@
 F 2 "audio-fx:Potentiometer_Alps_RK09L_Single_Vertical" H 1650 5800 50  0001 C CNN
 F 3 "~" H 1650 5800 50  0001 C CNN
+F 4 "729-3600" H 1650 5800 50  0001 C CNN "rs"
 	1    1650 5800
 	1    0    0    -1
@@
 F 2 "audio-fx:Potentiometer_Alps_RK09L_Single_Vertical" H 2400 5800 50  0001 C CNN
 F 3 "~" H 2400 5800 50  0001 C CNN
+F 4 "729-3600" H 2400 5800 50  0001 C CNN "rs"
 	1    2400 5800
 	1    0    0    -1
@@
 F 2 "audio-fx:Potentiometer_Alps_RK09L_Single_Vertical" H 3150 5800 50  0001 C CNN
 F 3 "~" H 3150 5800 50  0001 C CNN
+F 4 "729-3600" H 3150 5800 50  0001 C CNN "rs"
 	1    3150 5800
 	1    0    0    -1
@@
 F 2 "audio-fx:Potentiometer_Alps_RK09L_Single_Vertical" H 3900 5800 50  0001 C CNN
 F 3 "~" H 3900 5800 50  0001 C CNN
+F 4 "729-3600" H 3900 5800 50  0001 C CNN "rs"
 	1    3900 5800
 	1    0    0    -1
@@
 F 2 "audio-fx:Potentiometer_Alps_RK09L_Single_Vertical" H 1650 6750 50  0001 C CNN
 F 3 "~" H 1650 6750 50  0001 C CNN
+F 4 "729-3600" H 1650 6750 50  0001 C CNN "rs"
 	1    1650 6750
 	1    0    0    -1
@@
 F 2 "audio-fx:Potentiometer_Alps_RK09L_Single_Vertical" H 2400 6750 50  0001 C CNN
 F 3 "~" H 2400 6750 50  0001 C CNN
+F 4 "729-3600" H 2400 6750 50  0001 C CNN "rs"
 	1    2400 6750
 	1    0    0    -1
@@
 F 2 "audio-fx:Potentiometer_Alps_RK09L_Single_Vertical" H 3150 6750 50  0001 C CNN
 F 3 "~" H 3150 6750 50  0001 C CNN
+F 4 "729-3600" H 3150 6750 50  0001 C CNN "rs"
 	1    3150 6750
 	1    0    0    -1
@@
 F 2 "audio-fx:Potentiometer_Alps_RK09L_Single_Vertical" H 3900 6750 50  0001 C CNN
 F 3 "~" H 3900 6750 50  0001 C CNN
+F 4 "729-3600" H 3900 6750 50  0001 C CNN "rs"
 	1    3900 6750
 	1    0    0    -1
@@
 F 2 "Capacitor_SMD:C_0805_2012Metric" H 3638 1550 50  0001 C CNN
 F 3 "~" H 3600 1700 50  0001 C CNN
+F 4 "2773238" H 3600 1700 50  0001 C CNN "farnell"
 	1    3600 1700
 	1    0    0    -1
@@
 F 2 "Button_Switch_THT:SW_PUSH_6mm" H 1600 2350 50  0001 C CNN
 F 3 "" H 1600 2350 50  0001 C CNN
+F 4 "dnp" H 1600 2150 50  0001 C CNN "farnell"
 	1    1600 2150
 	1    0    0    -1
@@
 F 2 "Button_Switch_THT:SW_PUSH_6mm" H 1600 2800 50  0001 C CNN
 F 3 "" H 1600 2800 50  0001 C CNN
+F 4 "dnp" H 1600 2600 50  0001 C CNN "farnell"
 	1    1600 2600
 	1    0    0    -1
@@
 F 2 "Button_Switch_THT:SW_PUSH_6mm" H 1600 3200 50  0001 C CNN
 F 3 "" H 1600 3200 50  0001 C CNN
+F 4 "dnp" H 1600 3000 50  0001 C CNN "farnell"
 	1    1600 3000
 	1    0    0    -1
@@
 F 2 "Button_Switch_THT:SW_PUSH_6mm" H 1600 3600 50  0001 C CNN
 F 3 "" H 1600 3600 50  0001 C CNN
+F 4 "dnp" H 1600 3400 50  0001 C CNN "farnell"
 	1    1600 3400
 	1    0    0    -1
@@
 P 6100 3300
 F 0 "R5" V 5893 3300 50  0000 C CNN
-F 1 "5k" V 5984 3300 50  0000 C CNN
+F 1 "4.7k" V 5984 3300 50  0000 C CNN
 F 2 "Resistor_SMD:R_0805_2012Metric" V 6030 3300 50  0001 C CNN
 F 3 "~" H 6100 3300 50  0001 C CNN
+F 4 "1469923" H 6100 3300 50  0001 C CNN "farnell"
 	1    6100 3300
 	0    1    1    0
@@
 F 2 "Capacitor_SMD:C_0805_2012Metric" H 5888 1950 50  0001 C CNN
 F 3 "~" H 5850 2100 50  0001 C CNN
+F 4 "2773238" H 5850 2100 50  0001 C CNN "farnell"
 	1    5850 2100
 	1    0    0    -1
@@
 F 2 "Capacitor_SMD:C_0805_2012Metric" H 9488 4950 50  0001 C CNN
 F 3 "~" H 9450 5100 50  0001 C CNN
+F 4 "2773238" H 9450 5100 50  0001 C CNN "farnell"
 	1    9450 5100
 	1    0    0    -1
@@
 F 2 "Inductor_SMD:L_0805_2012Metric" V 9180 4950 50  0001 C CNN
 F 3 "~" H 9250 4950 50  0001 C CNN
+F 4 "2215655" H 9250 4950 50  0001 C CNN "farnell"
 	1    9250 4950
 	0    -1   -1   0
@@
 P 3450 3400
 F 0 "R10" V 3243 3400 50  0000 C CNN
-F 1 "200r" V 3334 3400 50  0000 C CNN
+F 1 "100R" V 3334 3400 50  0000 C CNN
 F 2 "Resistor_SMD:R_0805_2012Metric" V 3380 3400 50  0001 C CNN
 F 3 "~" H 3450 3400 50  0001 C CNN
+F 4 "1469862" H 3450 3400 50  0001 C CNN "farnell"
 	1    3450 3400
 	0    1    1    0
@@
 F 2 "Capacitor_SMD:C_0805_2012Metric" H 3338 3400 50  0001 C CNN
 F 3 "~" H 3300 3550 50  0001 C CNN
-F 4 "" H 3300 3550 50  0001 C CNN "farnell"
+F 4 "2773238" H 3300 3550 50  0001 C CNN "farnell"
 	1    3300 3550
 	1    0    0    -1
@@
 Connection ~ 3300 3400
 Text Notes 2800 4150 0    50   ~ 0
-RC filter\n200R & 2.2u = 360Hz cutoff
+RC filter\n200R & 2.2u = 700Hz cutoff
 Text Notes 2200 7300 0    50   ~ 0
 all pots 10k, taper 1b (linear)\nRK09K1130AP5
