File: hardware/pots.sch (KiCad schematic (older format))
At the start: 46 parts, among them SW1 Switch_SW_Push, SW2 Switch_SW_Push, SW3 Switch_SW_Push, SW4 Switch_SW_Push, U4 4067, U5 TLC5947DAP

Commit message: change farnell field to farnell #
Parts:
- C10, C11, C12, C16: farnell 2773238 -> (none); farnell # (none) -> 2773238
- D1, D10, D11, D12, D13, D14, D15, D16, D17, D18, D19, D2, D20, D3, D4, D5, D6, D7, D8, D9: farnell 2099236 -> (none); farnell # (none) -> 2099236
- L2: farnell 2215655 -> (none); farnell # (none) -> 2215655
- R10: farnell 1469862 -> (none); farnell # (none) -> 1469862
- R4: farnell 2906645 -> (none); farnell # (none) -> 2906645
- R5: farnell 1469923 -> (none); farnell # (none) -> 1469923
- SW1, SW2, SW3, SW4: farnell dnp -> (none); farnell # (none) -> dnp
- U4: farnell 3124957 -> (none); farnell # (none) -> 3124957
- U5: farnell 1755259 -> (none); farnell # (none) -> 1755259
Changed lines of the file:
@@
 F 2 "audio-fx:Potentiometer_Alps_RK09L_Single_Vertical" H 1650 4900 50  0001 C CNN
 F 3 "https://docs.rs-online.com/06f8/0900766b80f4c571.pdf" H 1650 4900 50  0001 C CNN
-F 4 "" H 1650 4900 50  0001 C CNN "farnell"
+F 4 "" H 1650 4900 50  0001 C CNN "farnell #"
 F 5 "729-3600" H 1650 4900 50  0001 C CNN "rs"
 	1    1650 4900
@@
 F 2 "Resistor_SMD:R_0805_2012Metric" V 3380 2300 50  0001 C CNN
 F 3 "~" H 3450 2300 50  0001 C CNN
-F 4 "2906645" H 3450 2300 50  0001 C CNN "farnell"
+F 4 "2906645" H 3450 2300 50  0001 C CNN "farnell #"
 	1    3450 2300
 	0    1    1    0
@@
 F 2 "Package_SO:SSOP-24_5.3x8.2mm_P0.65mm" H 4200 2850 50  0001 C CNN
 F 3 "https://www.ti.com/lit/ds/symlink/cd74hc4067.pdf" H 4200 2850 50  0001 C CNN
-F 4 "3124957" H 4200 2850 50  0001 C CNN "farnell"
+F 4 "3124957" H 4200 2850 50  0001 C CNN "farnell #"
 	1    4200 2850
 	1    0    0    -1
@@
 F 2 "Capacitor_SMD:C_0805_2012Metric" H 3638 1550 50  0001 C CNN
 F 3 "~" H 3600 1700 50  0001 C CNN
-F 4 "2773238" H 3600 1700 50  0001 C CNN "farnell"
+F 4 "2773238" H 3600 1700 50  0001 C CNN "farnell #"
 	1    3600 1700
 	1    0    0    -1
@@
 F 2 "Button_Switch_THT:SW_PUSH_6mm" H 1600 2350 50  0001 C CNN
 F 3 "" H 1600 2350 50  0001 C CNN
-F 4 "dnp" H 1600 2150 50  0001 C CNN "farnell"
+F 4 "dnp" H 1600 2150 50  0001 C CNN "farnell #"
 	1    1600 2150
 	1    0    0    -1
@@
 F 2 "Button_Switch_THT:SW_PUSH_6mm" H 1600 2800 50  0001 C CNN
 F 3 "" H 1600 2800 50  0001 C CNN
-F 4 "dnp" H 1600 2600 50  0001 C CNN "farnell"
+F 4 "dnp" H 1600 2600 50  0001 C CNN "farnell #"
 	1    1600 2600
 	1    0    0    -1
@@
 F 2 "Button_Switch_THT:SW_PUSH_6mm" H 1600 3200 50  0001 C CNN
 F 3 "" H 1600 3200 50  0001 C CNN
-F 4 "dnp" H 1600 3000 50  0001 C CNN "farnell"
+F 4 "dnp" H 1600 3000 50  0001 C CNN "farnell #"
 	1    1600 3000
 	1    0    0    -1
@@
 F 2 "Button_Switch_THT:SW_PUSH_6mm" H 1600 3600 50  0001 C CNN
 F 3 "" H 1600 3600 50  0001 C CNN
-F 4 "dnp" H 1600 3400 50  0001 C CNN "farnell"
+F 4 "dnp" H 1600 3400 50  0001 C CNN "farnell #"
 	1    1600 3400
 	1    0    0    -1
@@
 F 2 "LED_SMD:LED_0805_2012Metric" H 9400 3000 50  0001 C CNN
 F 3 "~" H 9400 3000 50  0001 C CNN
-F 4 "2099236" H 9400 3000 50  0001 C CNN "farnell"
+F 4 "2099236" H 9400 3000 50  0001 C CNN "farnell #"
 	1    9400 3000
 	1    0    0    -1
@@
 F 2 "LED_SMD:LED_0805_2012Metric" H 8800 2900 50  0001 C CNN
 F 3 "~" H 8800 2900 50  0001 C CNN
-F 4 "2099236" H 8800 2900 50  0001 C CNN "farnell"
+F 4 "2099236" H 8800 2900 50  0001 C CNN "farnell #"
 	1    8800 2900
 	1    0    0    -1
@@
 F 2 "LED_SMD:LED_0805_2012Metric" H 8250 2800 50  0001 C CNN
 F 3 "~" H 8250 2800 50  0001 C CNN
-F 4 "2099236" H 8250 2800 50  0001 C CNN "farnell"
+F 4 "2099236" H 8250 2800 50  0001 C CNN "farnell #"
 	1    8250 2800
 	1    0    0    -1
@@
 F 2 "LED_SMD:LED_0805_2012Metric" H 10000 2700 50  0001 C CNN
 F 3 "~" H 10000 2700 50  0001 C CNN
-F 4 "2099236" H 10000 2700 50  0001 C CNN "farnell"
+F 4 "2099236" H 10000 2700 50  0001 C CNN "farnell #"
 	1    10000 2700
 	1    0    0    -1
@@
 F 2 "LED_SMD:LED_0805_2012Metric" H 9400 2600 50  0001 C CNN
 F 3 "~" H 9400 2600 50  0001 C CNN
-F 4 "2099236" H 9400 2600 50  0001 C CNN "farnell"
+F 4 "2099236" H 9400 2600 50  0001 C CNN "farnell #"
 	1    9400 2600
 	1    0    0    -1
@@
 F 2 "LED_SMD:LED_0805_2012Metric" H 8800 2500 50  0001 C CNN
 F 3 "~" H 8800 2500 50  0001 C CNN
-F 4 "2099236" H 8800 2500 50  0001 C CNN "farnell"
+F 4 "2099236" H 8800 2500 50  0001 C CNN "farnell #"
 	1    8800 2500
 	1    0    0    -1
@@
 F 2 "LED_SMD:LED_0805_2012Metric" H 8250 2400 50  0001 C CNN
 F 3 "~" H 8250 2400 50  0001 C CNN
-F 4 "2099236" H 8250 2400 50  0001 C CNN "farnell"
+F 4 "2099236" H 8250 2400 50  0001 C CNN "farnell #"
 	1    8250 2400
 	1    0    0    -1
@@
 F 2 "Package_SO:HTSSOP-32-1EP_6.1x11mm_P0.65mm_EP5.2x11mm_Mask4.11x4.36mm" H 6400 5200 50  0001 L CNN
 F 3 "http://www.ti.com/lit/ds/symlink/tlc5947.pdf" H 6950 3600 50  0001 C CNN
-F 4 "1755259" H 6950 3600 50  0001 C CNN "farnell"
+F 4 "1755259" H 6950 3600 50  0001 C CNN "farnell #"
 	1    6950 3600
 	1    0    0    -1
@@
 F 2 "LED_SMD:LED_0805_2012Metric" H 10000 3100 50  0001 C CNN
 F 3 "~" H 10000 3100 50  0001 C CNN
-F 4 "2099236" H 10000 3100 50  0001 C CNN "farnell"
+F 4 "2099236" H 10000 3100 50  0001 C CNN "farnell #"
 	1    10000 3100
 	1    0    0    -1
@@
 F 2 "LED_SMD:LED_0805_2012Metric" H 9400 3800 50  0001 C CNN
 F 3 "~" H 9400 3800 50  0001 C CNN
-F 4 "2099236" H 9400 3800 50  0001 C CNN "farnell"
+F 4 "2099236" H 9400 3800 50  0001 C CNN "farnell #"
 	1    9400 3800
 	1    0    0    -1
@@
 F 2 "LED_SMD:LED_0805_2012Metric" H 8800 3700 50  0001 C CNN
 F 3 "~" H 8800 3700 50  0001 C CNN
-F 4 "2099236" H 8800 3700 50  0001 C CNN "farnell"
+F 4 "2099236" H 8800 3700 50  0001 C CNN "farnell #"
 	1    8800 3700
 	1    0    0    -1
@@
 F 2 "LED_SMD:LED_0805_2012Metric" H 8250 3600 50  0001 C CNN
 F 3 "~" H 8250 3600 50  0001 C CNN
-F 4 "2099236" H 8250 3600 50  0001 C CNN "farnell"
+F 4 "2099236" H 8250 3600 50  0001 C CNN "farnell #"
 	1    8250 3600
 	1    0    0    -1
@@
 F 2 "LED_SMD:LED_0805_2012Metric" H 10000 3500 50  0001 C CNN
 F 3 "~" H 10000 3500 50  0001 C CNN
-F 4 "2099236" H 10000 3500 50  0001 C CNN "farnell"
+F 4 "2099236" H 10000 3500 50  0001 C CNN "farnell #"
 	1    10000 3500
 	1    0    0    -1
@@
 F 2 "LED_SMD:LED_0805_2012Metric" H 9400 3400 50  0001 C CNN
 F 3 "~" H 9400 3400 50  0001 C CNN
-F 4 "2099236" H 9400 3400 50  0001 C CNN "farnell"
+F 4 "2099236" H 9400 3400 50  0001 C CNN "farnell #"
 	1    9400 3400
 	1    0    0    -1
@@
 F 2 "LED_SMD:LED_0805_2012Metric" H 8800 3300 50  0001 C CNN
 F 3 "~" H 8800 3300 50  0001 C CNN
-F 4 "2099236" H 8800 3300 50  0001 C CNN "farnell"
+F 4 "2099236" H 8800 3300 50  0001 C CNN "farnell #"
 	1    8800 3300
 	1    0    0    -1
@@
 F 2 "LED_SMD:LED_0805_2012Metric" H 8250 3200 50  0001 C CNN
 F 3 "~" H 8250 3200 50  0001 C CNN
-F 4 "2099236" H 8250 3200 50  0001 C CNN "farnell"
+F 4 "2099236" H 8250 3200 50  0001 C CNN "farnell #"
 	1    8250 3200
 	1    0    0    -1
@@
 F 2 "LED_SMD:LED_0805_2012Metric" H 10000 3900 50  0001 C CNN
 F 3 "~" H 10000 3900 50  0001 C CNN
-F 4 "2099236" H 10000 3900 50  0001 C CNN "farnell"
+F 4 "2099236" H 10000 3900 50  0001 C CNN "farnell #"
 	1    10000 3900
 	1    0    0    -1
@@
 F 2 "Resistor_SMD:R_0805_2012Metric" V 6030 3300 50  0001 C CNN
 F 3 "~" H 6100 3300 50  0001 C CNN
-F 4 "1469923" H 6100 3300 50  0001 C CNN "farnell"
+F 4 "1469923" H 6100 3300 50  0001 C CNN "farnell #"
 	1    6100 3300
 	0    1    1    0
@@
 F 2 "Capacitor_SMD:C_0805_2012Metric" H 5888 1950 50  0001 C CNN
 F 3 "~" H 5850 2100 50  0001 C CNN
-F 4 "2773238" H 5850 2100 50  0001 C CNN "farnell"
+F 4 "2773238" H 5850 2100 50  0001 C CNN "farnell #"
 	1    5850 2100
 	1    0    0    -1
@@
 F 2 "Capacitor_SMD:C_0805_2012Metric" H 9488 4950 50  0001 C CNN
 F 3 "~" H 9450 5100 50  0001 C CNN
-F 4 "2773238" H 9450 5100 50  0001 C CNN "farnell"
+F 4 "2773238" H 9450 5100 50  0001 C CNN "farnell #"
 	1    9450 5100
 	1    0    0    -1
@@
 F 2 "Inductor_SMD:L_0805_2012Metric" V 9180 4950 50  0001 C CNN
 F 3 "~" H 9250 4950 50  0001 C CNN
-F 4 "2215655" H 9250 4950 50  0001 C CNN "farnell"
+F 4 "2215655" H 9250 4950 50  0001 C CNN "farnell #"
 	1    9250 4950
 	0    -1   -1   0
@@
 F 2 "LED_SMD:LED_0805_2012Metric" H 9400 4200 50  0001 C CNN
 F 3 "~" H 9400 4200 50  0001 C CNN
-F 4 "2099236" H 9400 4200 50  0001 C CNN "farnell"
+F 4 "2099236" H 9400 4200 50  0001 C CNN "farnell #"
 	1    9400 4200
 	1    0    0    -1
@@
 F 2 "LED_SMD:LED_0805_2012Metric" H 8800 4100 50  0001 C CNN
 F 3 "~" H 8800 4100 50  0001 C CNN
-F 4 "2099236" H 8800 4100 50  0001 C CNN "farnell"
+F 4 "2099236" H 8800 4100 50  0001 C CNN "farnell #"
 	1    8800 4100
 	1    0    0    -1
@@
 F 2 "LED_SMD:LED_0805_2012Metric" H 8250 4000 50  0001 C CNN
 F 3 "~" H 8250 4000 50  0001 C CNN
-F 4 "2099236" H 8250 4000 50  0001 C CNN "farnell"
+F 4 "2099236" H 8250 4000 50  0001 C CNN "farnell #"
 	1    8250 4000
 	1    0    0    -1
@@
 F 2 "LED_SMD:LED_0805_2012Metric" H 10000 4300 50  0001 C CNN
 F 3 "~" H 10000 4300 50  0001 C CNN
-F 4 "2099236" H 10000 4300 50  0001 C CNN "farnell"
+F 4 "2099236" H 10000 4300 50  0001 C CNN "farnell #"
 	1    10000 4300
 	1    0    0    -1
@@
 F 2 "Resistor_SMD:R_0805_2012Metric" V 3380 3400 50  0001 C CNN
 F 3 "~" H 3450 3400 50  0001 C CNN
-F 4 "1469862" H 3450 3400 50  0001 C CNN "farnell"
+F 4 "1469862" H 3450 3400 50  0001 C CNN "farnell #"
 	1    3450 3400
 	0    1    1    0
@@
 F 2 "Capacitor_SMD:C_0805_2012Metric" H 3338 3400 50  0001 C CNN
 F 3 "~" H 3300 3550 50  0001 C CNN
-F 4 "2773238" H 3300 3550 50  0001 C CNN "farnell"
+F 4 "2773238" H 3300 3550 50  0001 C CNN "farnell #"
 	1    3300 3550
 	1    0    0    -1

Commit message: fix library mess and get bom exported
Parts:
- SW1, SW2, SW3, SW4: symbol teensy-fx-rescue:Switch_SW_Push-teensy_beats-cache -> teensy-fx:Switch_SW_Push-teensy_beats-cache
- U4: symbol teensy-fx-rescue:4067-teensy_beats-cache -> teensy-fx:4067-teensy_beats-cache
Changed lines of the file:
@@
 $EndComp
 $Comp
-L teensy-fx-rescue:4067-teensy_beats-cache U4
+L teensy-fx:4067-teensy_beats-cache U4
 U 1 1 5E1AC48F
 P 4200 2850
@@
 $EndComp
 $Comp
-L teensy-fx-rescue:Switch_SW_Push-teensy_beats-cache SW1
+L teensy-fx:Switch_SW_Push-teensy_beats-cache SW1
 U 1 1 5E252246
 P 1600 2150
@@
 $EndComp
 $Comp
-L teensy-fx-rescue:Switch_SW_Push-teensy_beats-cache SW2
+L teensy-fx:Switch_SW_Push-teensy_beats-cache SW2
 U 1 1 5E252D7C
 P 1600 2600
@@
 $EndComp
 $Comp
-L teensy-fx-rescue:Switch_SW_Push-teensy_beats-cache SW3
+L teensy-fx:Switch_SW_Push-teensy_beats-cache SW3
 U 1 1 5E2538C8
 P 1600 3000
@@
 $EndComp
 $Comp
-L teensy-fx-rescue:Switch_SW_Push-teensy_beats-cache SW4
+L teensy-fx:Switch_SW_Push-teensy_beats-cache SW4
 U 1 1 5E253CCE
 P 1600 3400

Commit message: cheaper caps and non-us 10k resistor
Parts:
- C10, C11, C12, C16: farnell # 2773238 -> 1759424
- R4: farnell # 2906645 -> 1469856
Changed lines of the file:
@@
 F 2 "Resistor_SMD:R_0805_2012Metric" V 3380 2300 50  0001 C CNN
 F 3 "~" H 3450 2300 50  0001 C CNN
-F 4 "2906645" H 3450 2300 50  0001 C CNN "farnell #"
+F 4 "1469856" H 3450 2300 50  0001 C CNN "farnell #"
 	1    3450 2300
 	0    1    1    0
@@
 F 2 "Capacitor_SMD:C_0805_2012Metric" H 3638 1550 50  0001 C CNN
 F 3 "~" H 3600 1700 50  0001 C CNN
-F 4 "2773238" H 3600 1700 50  0001 C CNN "farnell #"
+F 4 "1759424" H 3600 1700 50  0001 C CNN "farnell #"
 	1    3600 1700
 	1    0    0    -1
@@
 F 2 "Capacitor_SMD:C_0805_2012Metric" H 5888 1950 50  0001 C CNN
 F 3 "~" H 5850 2100 50  0001 C CNN
-F 4 "2773238" H 5850 2100 50  0001 C CNN "farnell #"
+F 4 "1759424" H 5850 2100 50  0001 C CNN "farnell #"
 	1    5850 2100
 	1    0    0    -1
@@
 F 2 "Capacitor_SMD:C_0805_2012Metric" H 9488 4950 50  0001 C CNN
 F 3 "~" H 9450 5100 50  0001 C CNN
-F 4 "2773238" H 9450 5100 50  0001 C CNN "farnell #"
+F 4 "1759424" H 9450 5100 50  0001 C CNN "farnell #"
 	1    9450 5100
 	1    0    0    -1
@@
 F 2 "Capacitor_SMD:C_0805_2012Metric" H 3338 3400 50  0001 C CNN
 F 3 "~" H 3300 3550 50  0001 C CNN
-F 4 "2773238" H 3300 3550 50  0001 C CNN "farnell #"
+F 4 "1759424" H 3300 3550 50  0001 C CNN "farnell #"
 	1    3300 3550
 	1    0    0    -1

Commit message: add farnell number for switches
Parts:
- SW1, SW2, SW3, SW4: farnell # dnp -> 1608274
Changed lines of the file:
@@
 F 2 "Button_Switch_THT:SW_PUSH_6mm" H 1600 2350 50  0001 C CNN
 F 3 "" H 1600 2350 50  0001 C CNN
-F 4 "dnp" H 1600 2150 50  0001 C CNN "farnell #"
+F 4 "1608274" H 1600 2150 50  0001 C CNN "farnell #"
 	1    1600 2150
 	1    0    0    -1
@@
 F 2 "Button_Switch_THT:SW_PUSH_6mm" H 1600 2800 50  0001 C CNN
 F 3 "" H 1600 2800 50  0001 C CNN
-F 4 "dnp" H 1600 2600 50  0001 C CNN "farnell #"
+F 4 "1608274" H 1600 2600 50  0001 C CNN "farnell #"
 	1    1600 2600
 	1    0    0    -1
@@
 F 2 "Button_Switch_THT:SW_PUSH_6mm" H 1600 3200 50  0001 C CNN
 F 3 "" H 1600 3200 50  0001 C CNN
-F 4 "dnp" H 1600 3000 50  0001 C CNN "farnell #"
+F 4 "1608274" H 1600 3000 50  0001 C CNN "farnell #"
 	1    1600 3000
 	1    0    0    -1
@@
 F 2 "Button_Switch_THT:SW_PUSH_6mm" H 1600 3600 50  0001 C CNN
 F 3 "" H 1600 3600 50  0001 C CNN
-F 4 "dnp" H 1600 3400 50  0001 C CNN "farnell #"
+F 4 "1608274" H 1600 3400 50  0001 C CNN "farnell #"
 	1    1600 3400
 	1    0    0    -1

Commit message: fix wiring & routing for lrclk and bclk, and removed lp filter behind pot mux
Parts:
- removed C16: 2.2uF, Capacitor_SMD:C_0805_2012Metric, symbol Device:C
- removed R10: 100R, Resistor_SMD:R_0805_2012Metric, symbol Device:R
Connections:
- wire segments 57 -> 56
Other:
- note removed: "RC filter\n200R & 2.2u = 700Hz cutoff"
Changed lines of the file:
@@
 encoding utf-8
 Sheet 3 3
-Title ""
-Date ""
-Rev ""
-Comp ""
+Title "teensy-fx"
+Date "2020-02-10"
+Rev "v2"
+Comp "mattvenn"
 Comment1 ""
 Comment2 ""
@@
 	1    0    0    -1
 $EndComp
-Text GLabel 3250 3400 0    50   Input ~ 0
+Text GLabel 3600 3400 0    50   Input ~ 0
 pot_multiplex
 Text GLabel 3600 2700 0    50   Input ~ 0
@@
 Wire Wire Line
 	10150 4200 10150 4100
-$Comp
-L Device:R R10
-U 1 1 5E14FB1F
-P 3450 3400
-F 0 "R10" V 3243 3400 50  0000 C CNN
-F 1 "100R" V 3334 3400 50  0000 C CNN
-F 2 "Resistor_SMD:R_0805_2012Metric" V 3380 3400 50  0001 C CNN
-F 3 "~" H 3450 3400 50  0001 C CNN
-F 4 "1469862" H 3450 3400 50  0001 C CNN "farnell #"
-	1    3450 3400
-	0    1    1    0
-$EndComp
-$Comp
-L Device:C C16
-U 1 1 5E1525F8
-P 3300 3550
-F 0 "C16" H 3415 3596 50  0000 L CNN
-F 1 "2.2uF" H 3415 3505 50  0000 L CNN
-F 2 "Capacitor_SMD:C_0805_2012Metric" H 3338 3400 50  0001 C CNN
-F 3 "~" H 3300 3550 50  0001 C CNN
-F 4 "1759424" H 3300 3550 50  0001 C CNN "farnell #"
-	1    3300 3550
-	1    0    0    -1
-$EndComp
-$Comp
-L power:GND #PWR0177
-U 1 1 5E1577D0
-P 3300 3700
-F 0 "#PWR0177" H 3300 3450 50  0001 C CNN
-F 1 "GND" H 3305 3527 50  0000 C CNN
-F 2 "" H 3300 3700 50  0001 C CNN
-F 3 "" H 3300 3700 50  0001 C CNN
-	1    3300 3700
-	1    0    0    -1
-$EndComp
-Wire Wire Line
-	3250 3400 3300 3400
-Connection ~ 3300 3400
-Text Notes 2800 4150 0    50   ~ 0
-RC filter\n200R & 2.2u = 700Hz cutoff
 Text Notes 2200 7300 0    50   ~ 0
 all pots 10k, taper 1b (linear)\nRK09K1130AP5
