File: hardware/teensy-fx.sch (KiCad schematic (older format))
At the start: 12 parts, among them U1 Teensy4.0, U6 W25Q128JVS

Commit message: farnell numbers
Parts:
- R6, R7: farnell (none) -> 2906645
- TP1, TP2, TP3, TP4, TP5, TP6, TP7, TP8, U6: farnell (none) -> dnp
Changed lines of the file:
@@
 F 2 "Package_SO:SOIC-8_5.23x5.23mm_P1.27mm" H 2500 6850 50  0001 C CNN
 F 3 "http://www.winbond.com/resource-files/w25q128jv_dtr%20revc%2003272018%20plus.pdf" H 2500 6850 50  0001 C CNN
+F 4 "dnp" H 2500 6850 50  0001 C CNN "farnell"
 	1    2500 6850
 	1    0    0    -1
@@
 F 2 "TestPoint:TestPoint_Pad_D1.0mm" H 9400 1700 50  0001 C CNN
 F 3 "~" H 9400 1700 50  0001 C CNN
+F 4 "dnp" H 9200 1700 50  0001 C CNN "farnell"
 	1    9200 1700
 	0    -1   -1   0
@@
 F 2 "TestPoint:TestPoint_Pad_D1.0mm" H 9400 2050 50  0001 C CNN
 F 3 "~" H 9400 2050 50  0001 C CNN
+F 4 "dnp" H 9200 2050 50  0001 C CNN "farnell"
 	1    9200 2050
 	0    -1   -1   0
@@
 F 2 "TestPoint:TestPoint_Pad_D1.0mm" H 9400 2400 50  0001 C CNN
 F 3 "~" H 9400 2400 50  0001 C CNN
+F 4 "dnp" H 9200 2400 50  0001 C CNN "farnell"
 	1    9200 2400
 	0    -1   -1   0
@@
 F 2 "TestPoint:TestPoint_Pad_D1.0mm" H 9400 2800 50  0001 C CNN
 F 3 "~" H 9400 2800 50  0001 C CNN
+F 4 "dnp" H 9200 2800 50  0001 C CNN "farnell"
 	1    9200 2800
 	0    -1   -1   0
@@
 F 2 "TestPoint:TestPoint_Pad_D1.0mm" H 10550 2050 50  0001 C CNN
 F 3 "~" H 10550 2050 50  0001 C CNN
+F 4 "dnp" H 10350 2050 50  0001 C CNN "farnell"
 	1    10350 2050
 	0    -1   -1   0
@@
 F 2 "TestPoint:TestPoint_Pad_D1.0mm" H 10550 1700 50  0001 C CNN
 F 3 "~" H 10550 1700 50  0001 C CNN
+F 4 "dnp" H 10350 1700 50  0001 C CNN "farnell"
 	1    10350 1700
 	0    -1   -1   0
@@
 F 2 "Resistor_SMD:R_0805_2012Metric" V 1180 6450 50  0001 C CNN
 F 3 "~" H 1250 6450 50  0001 C CNN
+F 4 "2906645" H 1250 6450 50  0001 C CNN "farnell"
 	1    1250 6450
 	0    1    1    0
@@
 F 2 "Resistor_SMD:R_0805_2012Metric" V 3080 6950 50  0001 C CNN
 F 3 "~" H 3150 6950 50  0001 C CNN
+F 4 "2906645" H 3150 6950 50  0001 C CNN "farnell"
 	1    3150 6950
 	0    1    1    0
@@
 F 2 "TestPoint:TestPoint_Pad_D1.0mm" H 10500 2800 50  0001 C CNN
 F 3 "~" H 10500 2800 50  0001 C CNN
+F 4 "dnp" H 10300 2800 50  0001 C CNN "farnell"
 	1    10300 2800
 	0    -1   -1   0
@@
 F 2 "TestPoint:TestPoint_Pad_D1.0mm" H 10500 2400 50  0001 C CNN
 F 3 "~" H 10500 2400 50  0001 C CNN
+F 4 "dnp" H 10300 2400 50  0001 C CNN "farnell"
 	1    10300 2400
 	0    -1   -1   0

Commit message: change farnell field to farnell #
Parts:
- R6, R7: farnell 2906645 -> (none); farnell # (none) -> 2906645
- TP1, TP2, TP3, TP4, TP5, TP6, TP7, TP8, U6: farnell dnp -> (none); farnell # (none) -> dnp
- U1: farnell 2847911 -> (none); farnell # (none) -> 2847911
Changed lines of the file:
@@
 F 1 "Teensy4.0" H 6100 4824 50  0000 C CNN
 F 2 "audio-fx:teensy4smt" H 5700 3500 50  0001 C CNN
-F 3 "https://uk.farnell.com/multicomp/2212sm-14g-75-b1-pcr/connector-rcpt-14pos-1row-2-54mm/dp/2847911" H 5700 3500 50  0001 C CNN
-F 4 "2847911" H 6100 3300 50  0001 C CNN "farnell"
+F 3 "https://uk.farnell #.com/multicomp/2212sm-14g-75-b1-pcr/connector-rcpt-14pos-1row-2-54mm/dp/2847911" H 5700 3500 50  0001 C CNN
+F 4 "2847911" H 6100 3300 50  0001 C CNN "farnell #"
 	1    6100 3300
 	1    0    0    -1
@@
 F 2 "Package_SO:SOIC-8_5.23x5.23mm_P1.27mm" H 2500 6850 50  0001 C CNN
 F 3 "http://www.winbond.com/resource-files/w25q128jv_dtr%20revc%2003272018%20plus.pdf" H 2500 6850 50  0001 C CNN
-F 4 "dnp" H 2500 6850 50  0001 C CNN "farnell"
+F 4 "dnp" H 2500 6850 50  0001 C CNN "farnell #"
 	1    2500 6850
 	1    0    0    -1
@@
 F 2 "TestPoint:TestPoint_Pad_D1.0mm" H 9400 1700 50  0001 C CNN
 F 3 "~" H 9400 1700 50  0001 C CNN
-F 4 "dnp" H 9200 1700 50  0001 C CNN "farnell"
+F 4 "dnp" H 9200 1700 50  0001 C CNN "farnell #"
 	1    9200 1700
 	0    -1   -1   0
@@
 F 2 "TestPoint:TestPoint_Pad_D1.0mm" H 9400 2050 50  0001 C CNN
 F 3 "~" H 9400 2050 50  0001 C CNN
-F 4 "dnp" H 9200 2050 50  0001 C CNN "farnell"
+F 4 "dnp" H 9200 2050 50  0001 C CNN "farnell #"
 	1    9200 2050
 	0    -1   -1   0
@@
 F 2 "TestPoint:TestPoint_Pad_D1.0mm" H 9400 2400 50  0001 C CNN
 F 3 "~" H 9400 2400 50  0001 C CNN
-F 4 "dnp" H 9200 2400 50  0001 C CNN "farnell"
+F 4 "dnp" H 9200 2400 50  0001 C CNN "farnell #"
 	1    9200 2400
 	0    -1   -1   0
@@
 F 2 "TestPoint:TestPoint_Pad_D1.0mm" H 9400 2800 50  0001 C CNN
 F 3 "~" H 9400 2800 50  0001 C CNN
-F 4 "dnp" H 9200 2800 50  0001 C CNN "farnell"
+F 4 "dnp" H 9200 2800 50  0001 C CNN "farnell #"
 	1    9200 2800
 	0    -1   -1   0
@@
 F 2 "TestPoint:TestPoint_Pad_D1.0mm" H 10550 2050 50  0001 C CNN
 F 3 "~" H 10550 2050 50  0001 C CNN
-F 4 "dnp" H 10350 2050 50  0001 C CNN "farnell"
+F 4 "dnp" H 10350 2050 50  0001 C CNN "farnell #"
 	1    10350 2050
 	0    -1   -1   0
@@
 F 2 "TestPoint:TestPoint_Pad_D1.0mm" H 10550 1700 50  0001 C CNN
 F 3 "~" H 10550 1700 50  0001 C CNN
-F 4 "dnp" H 10350 1700 50  0001 C CNN "farnell"
+F 4 "dnp" H 10350 1700 50  0001 C CNN "farnell #"
 	1    10350 1700
 	0    -1   -1   0
@@
 F 2 "Resistor_SMD:R_0805_2012Metric" V 1180 6450 50  0001 C CNN
 F 3 "~" H 1250 6450 50  0001 C CNN
-F 4 "2906645" H 1250 6450 50  0001 C CNN "farnell"
+F 4 "2906645" H 1250 6450 50  0001 C CNN "farnell #"
 	1    1250 6450
 	0    1    1    0
@@
 F 2 "Resistor_SMD:R_0805_2012Metric" V 3080 6950 50  0001 C CNN
 F 3 "~" H 3150 6950 50  0001 C CNN
-F 4 "2906645" H 3150 6950 50  0001 C CNN "farnell"
+F 4 "2906645" H 3150 6950 50  0001 C CNN "farnell #"
 	1    3150 6950
 	0    1    1    0
@@
 F 2 "TestPoint:TestPoint_Pad_D1.0mm" H 10500 2800 50  0001 C CNN
 F 3 "~" H 10500 2800 50  0001 C CNN
-F 4 "dnp" H 10300 2800 50  0001 C CNN "farnell"
+F 4 "dnp" H 10300 2800 50  0001 C CNN "farnell #"
 	1    10300 2800
 	0    -1   -1   0
@@
 F 2 "TestPoint:TestPoint_Pad_D1.0mm" H 10500 2400 50  0001 C CNN
 F 3 "~" H 10500 2400 50  0001 C CNN
-F 4 "dnp" H 10300 2400 50  0001 C CNN "farnell"
+F 4 "dnp" H 10300 2400 50  0001 C CNN "farnell #"
 	1    10300 2400
 	0    -1   -1   0

Commit message: cheaper caps and non-us 10k resistor
Parts:
- R6, R7: farnell # 2906645 -> 1469856
Changed lines of the file:
@@
 F 2 "Resistor_SMD:R_0805_2012Metric" V 1180 6450 50  0001 C CNN
 F 3 "~" H 1250 6450 50  0001 C CNN
-F 4 "2906645" H 1250 6450 50  0001 C CNN "farnell #"
+F 4 "1469856" H 1250 6450 50  0001 C CNN "farnell #"
 	1    1250 6450
 	0    1    1    0
@@
 F 2 "Resistor_SMD:R_0805_2012Metric" V 3080 6950 50  0001 C CNN
 F 3 "~" H 3150 6950 50  0001 C CNN
-F 4 "2906645" H 3150 6950 50  0001 C CNN "farnell #"
+F 4 "1469856" H 3150 6950 50  0001 C CNN "farnell #"
 	1    3150 6950
 	0    1    1    0
